Commit message: Optimized node, added yaw

File: radar_pose_detection/urdf/pile-setup-3d.urdf (robot description, URDF)
Before this commit: robot materials, 4 links, 2 joints
Joints:
- added joint base_to_pipe_z: type continuous, parent steel_pipe_y_dummy, child steel_pipe, origin xyz=0 0 0, axis 0 0 1
- joint base_to_pipe_y: axis 0 0 1 -> 0 1 0; child steel_pipe -> steel_pipe_y_dummy; parent steel_pipe_y_dummy -> steel_pipe_x_dummy

Commit message: Corrected frame of reference to be compatible with radar

File: radar_pose_detection/urdf/pile-setup-3d.urdf (robot description, URDF)
Before this commit: robot materials, 4 links, 3 joints
Links:
- removed link base_link
- added link ti_mmwave; visual box size=3 0.1 0.1
Joints:
- joint base_to_pipe_x: origin xyz=0 0 0 -> xyz=1 0 0.5; parent base_link -> ti_mmwave
