Commit message: Commented code

File: radar_pose_detection/urdf/pile-setup.urdf (robot description, URDF)
Before this commit: robot materials, 3 links, 2 joints
Links:
- removed link base_link
- added link ti_mmwave; visual box size=3 0.1 0.1
Joints:
- joint base_to_pipe_x: parent base_link -> ti_mmwave
